Commit message: add dg3f_b_driver & safety duty send

File: dg3f_b_driver/urdf/dg3f_b_ros2_control.xacro (robot description, xacro)
@@ -5,14 +5,14 @@
     <!-- prefix 변수 지정 -->
     <!-- <xacro:property name="prefix" value="${'rj' if hand == 'right' else 'lj'}"/> -->
-    <xacro:include filename="$(find dg_description)/urdf/dg3f_m.urdf"/>
+    <xacro:include filename="$(find dg_description)/urdf/dg3f_b.urdf"/>
     <link name="base_link" />
     <joint name="base_joint" type="fixed">
         <parent link="base_link"/>
-        <child link="l_dg_mount"/>
+        <child link="delto_base_link"/>
         <origin xyz="0 0 0" rpy="0 0 0"/>
     </joint>
-    <ros2_control name="dg3f_m_driver" type="system">
+    <ros2_control name="dg3f_b_driver" type="system">
         <hardware>
-            <plugin>dg3f_m_driver/SystemInterface</plugin>
+            <plugin>dg3f_b_driver/SystemInterface</plugin>
             <param name="delto_ip">$(arg delto_ip)</param>
             <param name="delto_port">$(arg delto_port)</param>
